File: hw/level2-1206.kicad_sch (KiCad schematic)
At the start: 6 parts, among them U2 LMC555xM, U6 USB_A, U7 1k

Commit message: Level 2 and 3
Parts:
- removed C4: 4.7u, Capacitor_SMD:C_1206_3216Metric_Pad1.33x1.80mm_HandSolder, symbol Device:C
- removed D2: LED, LED_SMD:LED_1206_3216Metric_Pad1.42x1.75mm_HandSolder, symbol Device:LED
- removed R4: 330R, Resistor_SMD:R_1206_3216Metric_Pad1.30x1.75mm_HandSolder, symbol Device:R
- removed U2: LMC555xM, Package_SO:SOIC-8_3.9x4.9mm_P1.27mm, symbol Timer:LMC555xM
- removed U6: USB_A, Robotarna_KiCad_Library:usb-PCB, symbol solderingChallenge-rescue:USB_A-Connector
- removed U7: 1k, Resistor_SMD:R_1206_3216Metric_Pad1.30x1.75mm_HandSolder, symbol Device:R
- added C?: 1u, Capacitor_SMD:C_1206_3216Metric_Pad1.33x1.80mm_HandSolder, symbol Device:C
- added D?: LED, LED_SMD:LED_1206_3216Metric_Pad1.42x1.75mm_HandSolder, symbol Device:LED
- added Klobouek?: redhatLogo, Robotarna_KiCad_Library:RedhatLogo, symbol Robotarna_KiCad_Library:redhatLogo
- added Kolecko?: robotarnaLogo, Robotarna_KiCad_Library:RobotarnaLogo-6mm, symbol Robotarna_KiCad_Library:robotarnaLogo
- added R? (x2): 470R, Resistor_SMD:R_1206_3216Metric_Pad1.30x1.75mm_HandSolder, symbol Device:R
- added R?: 1M, Resistor_SMD:R_1206_3216Metric_Pad1.30x1.75mm_HandSolder, symbol Device:R
- added U?: USB_A, Robotarna_KiCad_Library:usb-PCB, symbol solderingChallenge-rescue:USB_A-Connector
- added U?: LMC555xM, Package_SO:SOIC-8_3.9x4.9mm_P1.27mm, symbol Timer:LMC555xM
Connections:
- net GND: now also C?.2, R?.1, U?.1 (GND), U?.4 (GND)
- net VCC: now also R?.2, U?.1 (VBUS), U?.4 (R), U?.8 (VCC)
- new net: D?.1 (K), R?.1, R?.2
- new net: C?.1, R?.1, U?.2 (TR), U?.6 (THR)
- new net: D?.2 (A), R?.2, U?.3 (Q)
