File: hw/level3-0603.kicad_sch (KiCad schematic)
At the start: 6 parts, among them U3 LMC555xMM, U8 USB_A, U9 1k

Commit message: Level 2 and 3
Parts:
- removed C6: 4.7u, Capacitor_SMD:C_0603_1608Metric_Pad1.08x0.95mm_HandSolder, symbol Device:C
- removed D3: LED, LED_SMD:LED_0603_1608Metric_Pad1.05x0.95mm_HandSolder, symbol Device:LED
- removed R7: 330R, Resistor_SMD:R_0603_1608Metric_Pad1.05x0.95mm_HandSolder, symbol Device:R
- removed U3: LMC555xMM, Package_SO:VSSOP-8_3.0x3.0mm_P0.65mm, symbol Timer:LMC555xMM
- removed U8: USB_A, Robotarna_KiCad_Library:usb-PCB, symbol solderingChallenge-rescue:USB_A-Connector
- removed U9: 1k, Resistor_SMD:R_0603_1608Metric_Pad0.98x0.95mm_HandSolder, symbol Device:R
- added C?: 1uF, Capacitor_SMD:C_0603_1608Metric_Pad1.08x0.95mm_HandSolder, symbol Device:C
- added D?: LED, LED_SMD:LED_0603_1608Metric_Pad1.05x0.95mm_HandSolder, symbol Device:LED
- added Klobouek?: redhatLogo, Robotarna_KiCad_Library:RedhatLogo, symbol Robotarna_KiCad_Library:redhatLogo
- added Kolecko?: robotarnaLogo, Robotarna_KiCad_Library:RobotarnaLogo-6mm, symbol Robotarna_KiCad_Library:robotarnaLogo
- added R?: 1M, Resistor_SMD:R_0603_1608Metric_Pad0.98x0.95mm_HandSolder, symbol Device:R
- added R? (x2): 470, Resistor_SMD:R_0603_1608Metric_Pad0.98x0.95mm_HandSolder, symbol Device:R
- added U?: USB_A, Robotarna_KiCad_Library:usb-PCB, symbol solderingChallenge-rescue:USB_A-Connector
- added U?: LMC555xMM, Package_SO:VSSOP-8_3.0x3.0mm_P0.65mm, symbol Timer:LMC555xMM
Connections:
- net GND: now also C?.2, R?.2, U?.1 (GND), U?.4 (GND)
- net VCC: now also R?.1, U?.1 (VBUS), U?.4 (R), U?.8 (VCC)
- new net: C?.1, R?.2, U?.2 (TR), U?.6 (THR)
- new net: D?.1 (K), R?.1, R?.2
- new net: D?.2 (A), R?.1, U?.3 (Q)
